File: testKICAD/Make_FMU3_Power/FMU_Power/FMU_Power.kicad_pcb (KiCad board)
At the start: 2 copper layers, 12 x 15.2 mm, 13 parts, among them J1 Conn_01x02_Male, J2 Conn_01x04_Male, U1 MIC5332

Commit message: FMU power 수정본
Parts:
- J1: footprint Connector_PinHeader_2.54mm:PinHeader_1x02_P2.54mm_Vertical_SMD_Pin1Left -> wooslib:FMU3_VDD_5V_IN_Connector; moved to F.Cu
- J2: footprint Connector_PinHeader_2.54mm:PinHeader_1x04_P2.54mm_Vertical_SMD_Pin1Left -> wooslib:MIC5332_OUTPUT_Connector
- moved C2 85.6 mm to (151.8, 104.6)
- moved R1 85.1 mm to (155.1, 107.8)
- moved C3 85.0 mm to (156.9, 106.5)
- moved U1 84.9 mm to (153.2, 104.8)
- moved C4 84.7 mm to (156.5, 105.0)
- moved C5 84.6 mm to (157.0, 103.7)
- moved C1 84.6 mm to (149.2, 104.7)
- moved C6 84.4 mm to (156.0, 101.8)
- moved C7 83.9 mm to (155.2, 102.8)
- moved J2 83.8 mm to (154.3, 110.5)
- moved C8 83.4 mm to (155.3, 101.4)
- moved L1 83.3 mm to (146.8, 106.3)
- moved J1 80.2 mm to (145.7, 102.0), turned to 90 degrees
Routing:
- net /VDD_3V3_SENSORS: track 20.6 -> 25.2 mm, vias 0 -> 2
- net /FMU-VDD_3V3: track 14.7 -> 18.0 mm
- net /FMU-!RESET: track 9.14 -> 6.42 mm
- net /VDD_5V_IN: track 8.07 -> 6.19 mm, vias 1 -> 0
- net /VDD_3V3_SENSORS_EN: track 6.23 -> 4.81 mm
- net GND: track 14.6 -> 13.5 mm, vias 3 -> 0
- net Net-(C1-Pad1): track 9.44 -> 9.95 mm
Other:
- board size 12 x 15.2 mm -> 14 x 13 mm

Commit message: adding files
Routing:
- net /FMU-VDD_3V3: track 18.0 -> 10.1 mm, vias 2 -> 0
- net GND: track 13.5 -> 12.1 mm, vias 0 -> 2
- net /VDD_3V3_SENSORS: track 25.2 -> 24.9 mm, vias 2 -> 0
- removed copper zone on B.Cu, net GND
- removed copper zone on F.Cu, net GND
