File: testKICAD/FMU3_Power_make/FMU3_Power_make.sch (KiCad schematic (older format))
At the start: 13 parts, among them J1 Conn_01x03_Male, J2 Conn_01x04_Female, U1 MIC5332-SSYMT-TR

Commit message: save
Parts:
- removed L1: Kyocera KNH16C104bA5TS EMI filter, woos_FMU3:KNH16C104DA5TS_Filter, symbol Device:EMI_Filter_C
Connections:
- net VDD_5V_IN is gone; now on net FMU-VDD_5V5: J1.1 (Pin_1)
Changed lines of the file:
@@
 	3950 3350 3950 3950
-Wire Wire Line
-	3950 3950 3600 3950
 Wire Wire Line
 	3400 3950 3400 2700
@@
 Wire Wire Line
 	4300 2200 4300 2500
-$Comp
-L Device:EMI_Filter_C L1
-U 1 1 5EC9301C
-P 3600 2600
-F 0 "L1" H 3550 2900 50  0000 C CNN
-F 1 "Kyocera KNH16C104bA5TS EMI filter" H 3600 2800 50  0000 C CNN
-F 2 "woos_FMU3:KNH16C104DA5TS_Filter" V 3600 2600 50  0001 C CNN
-F 3 "http://www.murata.com/~/media/webrenewal/support/library/catalog/products/emc/emifil/c31e.ashx?la=en-gb" V 3600 2600 50  0001 C CNN
-F 4 "478-6878-1-ND" V 3500 2400 39  0000 C CNN "부품번호"
-	1    3600 2600
-	1    0    0    -1
-$EndComp
-Wire Wire Line
-	3800 2500 3950 2500
 Wire Wire Line
 	3250 1950 3250 2600
-Wire Wire Line
-	3600 2700 3600 3950
-Connection ~ 3600 3950
-Wire Wire Line
-	3600 3950 3400 3950
 Wire Wire Line
 	4800 2500 4650 2500
@@
 GND
 Wire Wire Line
-	2900 2500 3400 2500
-Wire Wire Line
 	2900 2600 3250 2600
 Wire Wire Line
@@
 Text Label 4500 2500 0    39   ~ 0
 FMU-VDD_5V5
+Wire Wire Line
+	2900 2500 3950 2500
+Wire Wire Line
+	3400 3950 3950 3950
 $EndSCHEMATC
