File: testKICAD/FMU3_Power_make/FMU3_Power_make.kicad_pcb (KiCad board)
At the start: 2 copper layers, 17.5 x 10.5 mm, 13 parts, among them J1 Conn_01x03_Male, J2 Conn_01x04_Female, U1 MIC5332-SSYMT-TR

Commit message: Parts 3D modelling
Parts:
- removed L1: Kyocera KNH16C104bA5TS EMI filter, woos_FMU3:KNH16C104DA5TS_Filter
- moved R1 9.32 mm to (107.5, 56.5)
- moved C1 8.16 mm to (106.0, 53.2), turned to 270 degrees
- moved J1 8.10 mm to (101.7, 49.9)
- moved C3 7.34 mm to (110.2, 57.2)
- moved U1 7.30 mm to (108.5, 54.2)
- moved C4 7.25 mm to (112.2, 54.0)
- moved C5 7.21 mm to (111.2, 56.0)
- moved C6 7.16 mm to (112.8, 56.9)
- moved J2 7.10 mm to (114.7, 49.9)
- moved C7 7.03 mm to (109.5, 51.4)
- moved C8 6.97 mm to (112.1, 51.3), turned to 0 degrees
- moved C2 6.75 mm to (107.0, 51.2), turned to 0 degrees
Connections:
- J1 pad 1: /VDD_5V_IN -> /FMU-VDD_5V5
Routing:
- net /FMU-VDD_5V5: track 7.61 -> 0.00 mm, vias 2 -> 0
- net /VDD_5V_IN: track 3.16 -> 0.00 mm
- net GND: track 17.6 -> 15.7 mm, vias 4 -> 3
- net /FMU-!RESET: track 13.6 -> 12.3 mm
- net Net-(C3-Pad1): track 2.34 -> 2.94 mm
- net /VDD_3V3_SENSORS_EN: track 9.73 -> 9.14 mm, vias 0 -> 2
Other:
- board size 17.5 x 10.5 mm -> 16.8 x 10.5 mm

Commit message: save
Other:
- board text added: "3V3_SENSORS"
- board text added: "FMU_3V3"
- board text added: "FMU_5V5"
- board text added: "FMU_RESET"
Changed lines of the file:
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@@
   (general
     (thickness 1.6)
-    (drawings 4)
+    (drawings 9)
     (tracks 49)
     (zones 0)
@@
     )
   )
+  (gr_text 3V3_SENSORS (at 103.37 54.59) (layer F.SilkS)
+    (effects (font (size 0.2 0.2) (thickness 0.05)))
+  )
+  (gr_text "FMU_5V5\n" (at 103.37 52.19) (layer F.SilkS)
+    (effects (font (size 0.2 0.2) (thickness 0.05)))
+  )
+  (gr_text "FMU_RESET\n" (at 116.27 57.04) (layer F.SilkS)
+    (effects (font (size 0.2 0.2) (thickness 0.05)))
+  )
+  (gr_text "FMU_3V3\n" (at 116.22 54.64) (layer F.SilkS)
+    (effects (font (size 0.2 0.2) (thickness 0.05)))
+  )
+  (gr_text 3V3_SENSORS (at 116.27 52.14) (layer F.SilkS)
+    (effects (font (size 0.2 0.2) (thickness 0.05)))
+  )
   (gr_line (start 101.5 60) (end 101.5 49.5) (layer Edge.Cuts) (width 0.05))
   (gr_line (start 118.25 60) (end 101.5 60) (layer Edge.Cuts) (width 0.05))
@@
   (segment (start 106.559998 53.63) (end 106.929998 54) (width 0.25) (layer F.Cu) (net 1))
   (segment (start 106 53.63) (end 106.559998 53.63) (width 0.25) (layer F.Cu) (net 1))
-  (segment (start 110.2 54.6) (end 110.2 56.2888) (width 0.25) (layer F.Cu) (net 2) (status 1000000))
-  (segment (start 109.47 54.5) (end 110.1 54.5) (width 0.25) (layer F.Cu) (net 2) (status 1000000))
-  (segment (start 110.1 54.5) (end 110.2 54.6) (width 0.25) (layer F.Cu) (net 2) (status 1000000))
-  (segment (start 110.2 56.2888) (end 110.2 56.7674) (width 0.25) (layer F.Cu) (net 2) (status 1000000))
+  (segment (start 110.2 54.6) (end 110.2 56.2888) (width 0.25) (layer F.Cu) (net 2))
+  (segment (start 109.47 54.5) (end 110.1 54.5) (width 0.25) (layer F.Cu) (net 2))
+  (segment (start 110.1 54.5) (end 110.2 54.6) (width 0.25) (layer F.Cu) (net 2))
+  (segment (start 110.2 56.2888) (end 110.2 56.7674) (width 0.25) (layer F.Cu) (net 2))
   (segment (start 111.3 55.47) (end 111.2 55.57) (width 0.25) (layer F.Cu) (net 3))
   (segment (start 111.3 54) (end 111.3 55.47) (width 0.25) (layer F.Cu) (net 3))
@@
   (segment (start 109.47 55.385) (end 107.915 56.94) (width 0.25) (layer F.Cu) (net 5))
   (segment (start 109.47 55) (end 109.47 55.385) (width 0.25) (layer F.Cu) (net 5))
-  (via (at 106.03 56.94) (size 0.8) (drill 0.4) (layers F.Cu B.Cu) (net 5))
-  (segment (start 107.51 56.94) (end 106.03 56.94) (width 0.25) (layer F.Cu) (net 5))
-  (via (at 103.4 54.549998) (size 0.8) (drill 0.4) (layers F.Cu B.Cu) (net 5))
-  (segment (start 106.03 56.94) (end 103.639998 54.549998) (width 0.25) (layer B.Cu) (net 5))
-  (segment (start 103.639998 54.549998) (end 103.4 54.549998) (width 0.25) (layer B.Cu) (net 5))
-  (segment (start 103.4 54.549998) (end 103.4 53.5) (width 0.25) (layer F.Cu) (net 5))
+  (segment (start 106.03 56.94) (end 103.639998 54.549998) (width 0.25) (layer B.Cu) (net 5) (status 1000000))
+  (segment (start 107.51 56.94) (end 106.03 56.94) (width 0.25) (layer F.Cu) (net 5) (status 1000000))
+  (segment (start 103.4 54.549998) (end 103.4 53.5) (width 0.25) (layer F.Cu) (net 5) (status 1000000))
+  (segment (start 103.639998 54.549998) (end 103.4 54.549998) (width 0.25) (layer B.Cu) (net 5) (status 1000000))
+  (via (at 103.4 54.549998) (size 0.8) (drill 0.4) (layers F.Cu B.Cu) (net 5) (status 1000000))
+  (via (at 106.03 56.94) (size 0.8) (drill 0.4) (layers F.Cu B.Cu) (net 5) (status 1000000))
   (via (at 114.34 55.95) (size 0.8) (drill 0.4) (layers F.Cu B.Cu) (net 6))
   (segment (start 116.25 55.95) (end 114.34 55.95) (width 0.25) (layer F.Cu) (net 6))

Commit message: FMU3_power gbr
Parts:
- moved R1 1.69 mm to (109.1, 57.1), turned to 180 degrees
- moved C5 1.61 mm to (112.8, 56.0), turned to 0 degrees
- moved C4 1.60 mm to (113.6, 54.6)
- moved C3 1.55 mm to (111.2, 56.1)
- moved J2 1.28 mm to (116.0, 49.9)
- moved C6 1.08 mm to (113.7, 57.6), turned to 0 degrees
- moved C1 0.84 mm to (106.5, 52.5), turned to 0 degrees
- moved C7 0.74 mm to (109.5, 52.1)
- moved C8 0.60 mm to (111.5, 51.3), turned to 90 degrees
- moved U1 0.56 mm to (108.5, 54.8)
- moved C2 0.28 mm to (106.9, 51.0)
- moved J1 0.12 mm to (101.6, 49.9)
Routing:
- net /FMU-VDD_5V5: track 0.00 -> 10.2 mm
- net /FMU-VDD_3V3: track 5.26 -> 11.8 mm
- net /VDD_3V3_SENSORS_EN: track 9.14 -> 12.8 mm
- net GND: track 15.7 -> 12.6 mm, vias 3 -> 4
- net /VDD_3V3_SENSORS: track 1.87 -> 0.00 mm
- net /FMU-!RESET: track 12.3 -> 13.7 mm
- net Net-(C3-Pad1): track 2.94 -> 1.97 mm
- removed copper zone on F.Cu, net /FMU-VDD_3V3
Other:
- board size 16.8 x 10.5 mm -> 18 x 10.5 mm
- board text added: "GND"

Commit message: save
Other:
- board text added: "3V3"
- board text added: "3V3_EN"
- board text added: "3V3_Sn"
- board text added: "5V5"
- board text added: "IN"
- board text added: "OUT"
- board text added: "RESET"
- board text removed: "3V3_SENSORS"
- board text removed: "FMU_3V3"
- board text removed: "FMU_5V5"
- board text removed: "FMU_RESET"
Changed lines of the file:
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@@
-(kicad_pcb (version 20171130) (host pcbnew "(5.1.6)-1")
+(kicad_pcb (version 20171130) (host pcbnew "(5.1.5)-3")
   (general
     (thickness 1.6)
-    (drawings 11)
+    (drawings 13)
     (tracks 54)
     (zones 0)
@@
   (page A4)
   (layers
-    (0 F.Cu signal hide)
-    (31 B.Cu signal hide)
+    (0 F.Cu signal)
+    (31 B.Cu signal)
     (32 B.Adhes user hide)
     (33 F.Adhes user hide)
-    (34 B.Paste user hide)
-    (35 F.Paste user hide)
+    (34 B.Paste user)
+    (35 F.Paste user)
     (36 B.SilkS user)
     (37 F.SilkS user)
-    (38 B.Mask user)
-    (39 F.Mask user)
+    (38 B.Mask user hide)
+    (39 F.Mask user hide)
     (40 Dwgs.User user hide)
     (41 Cmts.User user hide)
@@
     (44 Edge.Cuts user)
     (45 Margin user hide)
-    (46 B.CrtYd user)
-    (47 F.CrtYd user)
+    (46 B.CrtYd user hide)
+    (47 F.CrtYd user hide)
     (48 B.Fab user hide)
     (49 F.Fab user hide)
@@
     (at 109.51 52.14 90)
     (fp_text reference C7 (at 1 -0.425 180) (layer F.SilkS)
-      (effects (font (size 0.2 0.2) (thickness 0.05)))
+      (effects (font (size 0.4 0.4) (thickness 0.05)))
     )
     (fp_text value 0u1 (at 0.3 0.75 90) (layer F.Fab)
@@
     (at 109.08 57.09 180)
     (fp_text reference R1 (at 0.58 -0.6) (layer F.SilkS)
-      (effects (font (size 0.2 0.2) (thickness 0.05)))
+      (effects (font (size 0.4 0.4) (thickness 0.05)))
     )
     (fp_text value 10K (at 0.75 0.625) (layer F.Fab)
@@
     (at 112.81 55.98)
     (fp_text reference C5 (at 1.19 0.02) (layer F.SilkS)
-      (effects (font (size 0.2 0.2) (thickness 0.05)))
+      (effects (font (size 0.4 0.4) (thickness 0.05)))
     )
     (fp_text value 0u1 (at 0.3 0.75) (layer F.Fab)
@@
   (module woos_FMU3:Conn_01x04_SMD (layer F.Cu)
     (at 115.98 49.87)
-    (fp_text reference J2 (at 0.4 -0.1) (layer F.SilkS)
-      (effects (font (size 0.2 0.2) (thickness 0.05)))
+    (fp_text reference J2 (at -0.13 0.04) (layer F.SilkS)
+      (effects (font (size 0.4 0.4) (thickness 0.05)))
     )
     (fp_text value Conn_01x04_Female (at 1.3 9.9) (layer F.Fab)
@@
     (at 106.48 52.51)
     (fp_text reference C1 (at -0.7 0.74) (layer F.SilkS)
-      (effects (font (size 0.2 0.2) (thickness 0.05)))
+      (effects (font (size 0.4 0.4) (thickness 0.05)))
     )
     (fp_text value 0u1 (at 0.3 0.75) (layer F.Fab)
@@
     (at 106.91 50.98)
     (fp_text reference C2 (at -1.5 -1.15) (layer F.SilkS)
-      (effects (font (size 0.2 0.2) (thickness 0.05)))
+      (effects (font (size 0.4 0.4) (thickness 0.05)))
     )
     (fp_text value 10u/25V (at -0.5 1.2) (layer F.Fab)
@@
     (at 111.25 56.11 270)
     (fp_text reference C3 (at -1.05 0.4 180) (layer F.SilkS)
-      (effects (font (size 0.2 0.2) (thickness 0.05)))
+      (effects (font (size 0.4 0.4) (thickness 0.05)))
     )
     (fp_text value CC0402KRX7R7BB103 (at 0.3 0.75 90) (layer F.Fab)
@@
     (descr <b>CAPACITOR</b>)
     (fp_text reference C4 (at -1.55 -1) (layer F.SilkS)
-      (effects (font (size 0.2 0.2) (thickness 0.05)))
+      (effects (font (size 0.4 0.4) (thickness 0.05)))
     )
     (fp_text value 1u (at -0.625 1.025) (layer F.Fab)
@@
     (at 113.67 57.56)
     (fp_text reference C6 (at -1.42 1.19) (layer F.SilkS)
-      (effects (font (size 0.2 0.2) (thickness 0.05)))
+      (effects (font (size 0.4 0.4) (thickness 0.05)))
     )
     (fp_text value 22u/25V (at -0.525 1.3) (layer F.Fab)
@@
     (at 111.5 51.3 90)
     (fp_text reference C8 (at 1.3 -1.25 180) (layer F.SilkS)
-      (effects (font (size 0.2 0.2) (thickness 0.05)))
+      (effects (font (size 0.4 0.4) (thickness 0.05)))
     )
     (fp_text value 22u/25V (at -0.525 1.3 90) (layer F.Fab)
@@
   (module woos_FMU3:Conn_01x03_SMD (layer F.Cu)
     (at 101.58 49.89)
-    (fp_text reference J1 (at 0.5 -0.2) (layer F.SilkS)
-      (effects (font (size 0.2 0.2) (thickness 0.05)))
+    (fp_text reference J1 (at 0.26 0) (layer F.SilkS)
+      (effects (font (size 0.4 0.4) (thickness 0.05)))
     )
     (fp_text value Conn_01x03_Male (at 1.4 7.3) (layer F.Fab)
@@
   (module MIC5332-SSYMT-TR:SON50P200X200X60-9N (layer F.Cu)
     (at 108.55 54.81)
-    (fp_text reference U1 (at -1.4 -1.55) (layer F.SilkS)
-      (effects (font (size 0.2 0.2) (thickness 0.05)))
+    (fp_text reference U1 (at -0.83 -1.46) (layer F.SilkS)
+      (effects (font (size 0.4 0.4) (thickness 0.05)))
     )
     (fp_text value MIC5332-SSYMT-TR (at 0.3 1.7) (layer F.Fab)
@@
     )
   )
-  (gr_text GND (at 117.5 59.75) (layer F.SilkS)
-    (effects (font (size 0.2 0.2) (thickness 0.05)))
+  (gr_text OUT (at 117.47 49.84) (layer F.SilkS)
+    (effects (font (size 0.5 0.5) (thickness 0.05)))
+  )
+  (gr_text IN (at 103.25 49.85) (layer F.SilkS)
+    (effects (font (size 0.5 0.5) (thickness 0.05)))
+  )
+  (gr_text GND (at 117.5 59.59) (layer F.SilkS)
+    (effects (font (size 0.5 0.5) (thickness 0.05)))
   )
   (gr_text GND (at 103.25 57.25) (layer F.SilkS)
-    (effects (font (size 0.2 0.2) (thickness 0.05)))
+    (effects (font (size 0.5 0.5) (thickness 0.05)))
   )
   (gr_line (start 119.5 49.5) (end 119.5 60) (layer Edge.Cuts) (width 0.05))
-  (gr_text 3V3_SENSORS (at 103.37 54.75) (layer F.SilkS)
-    (effects (font (size 0.2 0.2) (thickness 0.05)))
-  )
-  (gr_text "FMU_5V5\n" (at 103.25 52.19) (layer F.SilkS)
-    (effects (font (size 0.2 0.2) (thickness 0.05)))
-  )
-  (gr_text "FMU_RESET\n" (at 117.5 57.25) (layer F.SilkS)
-    (effects (font (size 0.2 0.2) (thickness 0.05)))
-  )
-  (gr_text "FMU_3V3\n" (at 117.5 54.75) (layer F.SilkS)
-    (effects (font (size 0.2 0.2) (thickness 0.05)))
-  )
-  (gr_text 3V3_SENSORS (at 117.5 52.25) (layer F.SilkS)
-    (effects (font (size 0.2 0.2) (thickness 0.05)))
+  (gr_text 3V3_EN (at 103.32 54.74) (layer F.SilkS)
+    (effects (font (size 0.4 0.4) (thickness 0.05)))
+  )
+  (gr_text "5V5\n" (at 103.3 52.17) (layer F.SilkS)
+    (effects (font (size 0.5 0.5) (thickness 0.05)))
+  )
+  (gr_text "RESET\n" (at 117.5 57.25) (layer F.SilkS)
+    (effects (font (size 0.4 0.4) (thickness 0.05)))
+  )
+  (gr_text "3V3\n" (at 117.5 54.75) (layer F.SilkS)
+    (effects (font (size 0.5 0.5) (thickness 0.05)))
+  )
+  (gr_text 3V3_Sn (at 117.5 52.25) (layer F.SilkS)
+    (effects (font (size 0.4 0.4) (thickness 0.05)))
   )
   (gr_line (start 101.5 60) (end 101.5 49.5) (layer Edge.Cuts) (width 0.05))
