File: testKICAD/FMU3_Sensors_make/FMU3_Sensors_make.kicad_pcb (KiCad board)
At the start: 2 copper layers, 18.8 x 13.5 mm, 11 parts, among them J1 Conn_01x04, J2 Conn_01x05, U1 MPU-9250, U2 MS561101BA03-50, U3 ICM-20602

Commit message: save
Parts:
- J1: value Conn_01x04 -> Conn_01x05; footprint SENSOR_CONN:sensorconnect_1x4 -> SENSOR_CONN:sensorconnect_1x5
- moved J1 1.10 mm to (143.1, 41.4)
Connections:
- J1 pad 4: GND -> /MPU_DRDY
Routing:
- net /MPU_DRDY: track 0.00 -> 7.54 mm
- net /VDD_3V3_SENSORS: track 11.9 -> 10.6 mm
