File: testKICAD/sensormake_test/FMU3_Sensors_make.kicad_pcb (KiCad board)
At the start: 2 copper layers, 19.8 x 14.8 mm, 14 parts, among them J1 Conn_01x04, J2 Conn_01x05, U1 MPU-9250, U2 MS561101BA03-50, U3 ICM-20602

Commit message: save
Parts:
- J1: value Conn_01x04 -> Conn_01x05; footprint SENSOR_CONN:sensorconnect_1x4 -> SENSOR_CONN:sensorconnect_1x5
- moved C4 3.41 mm to (139.1, 44.3), turned to 270 degrees
- moved R1 2.25 mm to (147.8, 35.1), turned to 180 degrees
- moved C6 1.24 mm to (146.2, 40.8)
- moved J2 1.00 mm to (151.8, 40.2)
- moved U3 0.68 mm to (147.3, 43.3)
- moved C5 0.68 mm to (148.2, 40.9)
- moved U2 0.63 mm to (142.2, 45.8), turned to 0 degrees
- moved J1 0.16 mm to (135.8, 40.2)
Connections:
- J1 pad 4: GND -> /MPU_DRDY
Routing:
- net /MPU_DRDY: track 0.00 -> 13.6 mm, vias 0 -> 2
- net /BARO_CS: track 14.0 -> 19.7 mm
- net /ICM_CS: track 14.0 -> 18.7 mm
- net /SPI_INT_MOSI: track 24.8 -> 28.8 mm, vias 4 -> 3
- net /SPI_INT_MISO: track 19.8 -> 21.8 mm, vias 2 -> 3
- net /VDD_3V3_SENSORS: track 20.5 -> 18.7 mm, vias 2 -> 0
- net /SPI_INT_SCK: track 32.3 -> 30.8 mm, vias 4 -> 3
- net /MPU_CS: track 8.28 -> 7.74 mm
- net GND: track 28.4 -> 28.0 mm, vias 4 -> 3
Other:
- board size 19.8 x 14.8 mm -> 20 x 15.2 mm

Commit message: save Estimate
Parts:
- J1: value Conn_01x05 -> Conn_01x06_Male; footprint SENSOR_CONN:sensorconnect_1x5 -> SENSOR_CONN:sensorconnect_1x6
- moved J2 23.4 mm to (131.1, 29.2)
- moved C2 17.0 mm to (137.6, 24.8), turned to 270 degrees
- moved R1 16.8 mm to (134.4, 24.9), turned to 270 degrees
- moved C6 16.4 mm to (134.5, 29.3), turned to 90 degrees
- moved C1 15.4 mm to (135.9, 25.5), turned to 270 degrees
- moved C5 15.3 mm to (138.2, 29.3), turned to 90 degrees
- moved C4 15.2 mm to (142.6, 29.6), turned to 180 degrees
- moved U3 15.1 mm to (136.3, 32.9)
- moved C8 14.5 mm to (135.8, 28.6)
- moved J1 14.4 mm to (145.4, 29.5)
- moved U2 12.6 mm to (141.2, 33.2), turned to 270 degrees
- moved C3 12.1 mm to (140.2, 29.4), turned to 180 degrees
- moved C7 12.1 mm to (137.1, 29.3)
- moved U1 12.1 mm to (141.1, 25.5)
Connections:
- J1 pad 5: GND -> /ICM_DRDY
- U3 pad 6: Net-(U3-Pad6) -> /ICM_DRDY
Routing:
- net GND: track 28.0 -> 4.40 mm
- net /VDD_3V3_SENSORS: track 18.7 -> 42.1 mm, vias 0 -> 2
- net /SPI_INT_SCK: track 30.8 -> 9.94 mm, vias 3 -> 2
- net /SPI_INT_MOSI: track 28.8 -> 9.18 mm, vias 3 -> 2
- net /BARO_CS: track 19.7 -> 1.98 mm, vias 2 -> 1
- net /ICM_CS: track 18.7 -> 1.97 mm, vias 2 -> 1
- net /SPI_INT_MISO: track 21.8 -> 6.85 mm, vias 3 -> 1
- net /MPU_DRDY: track 13.6 -> 3.80 mm
- net /MPU_CS: track 7.74 -> 0.00 mm
- net /ICM_DRDY: track 0.00 -> 1.99 mm, vias 0 -> 1
- net Net-(C5-Pad1): track 1.09 -> 2.47 mm
- net (no net): vias 0 -> 2
- removed copper zone on F.Cu, net /VDD_3V3_SENSORS
- removed copper zone on B.Cu, net GND
- removed copper zone on F.Cu, net GND
Other:
- board outline removed

Commit message: save
Parts:
- moved C6 7.24 mm to (141.8, 28.7), turned to 0 degrees
- moved C4 6.99 mm to (135.6, 29.8), turned to 0 degrees
- moved C8 6.71 mm to (142.4, 30.0), turned to 0 degrees
- moved U3 6.43 mm to (142.6, 34.2)
- moved C5 5.66 mm to (143.5, 31.3), turned to 0 degrees
- moved C7 5.09 mm to (141.8, 31.3), turned to 0 degrees
- moved U2 4.08 mm to (137.3, 34.1), turned to 0 degrees
- moved C2 2.97 mm to (135.2, 26.7), turned to 180 degrees
- moved U1 2.28 mm to (138.8, 25.4)
- moved C3 2.10 mm to (138.2, 30.0)
- moved R1 1.38 mm to (135.1, 23.8), turned to 180 degrees
- moved C1 1.35 mm to (134.6, 25.3), turned to 180 degrees
- moved J1 0.48 mm to (145.0, 29.2)
Routing:
- net /VDD_3V3_SENSORS: track 42.1 -> 21.2 mm
- net GND: track 4.40 -> 24.5 mm, vias 3 -> 6
- net /BARO_CS: track 1.98 -> 19.4 mm, vias 1 -> 2
- net /SPI_INT_SCK: track 9.94 -> 25.4 mm, vias 2 -> 3
- net /SPI_INT_MOSI: track 9.18 -> 24.5 mm, vias 2 -> 3
- net /SPI_INT_MISO: track 6.85 -> 20.0 mm, vias 1 -> 3
- net /MPU_CS: track 0.00 -> 10.3 mm
- net /ICM_CS: track 1.97 -> 11.9 mm, vias 1 -> 2
- net /MPU_DRDY: track 3.80 -> 10.1 mm, vias 2 -> 0
- net /ICM_DRDY: track 1.99 -> 6.19 mm, vias 1 -> 0
- net Net-(C5-Pad1): track 2.47 -> 1.61 mm
- net Net-(C3-Pad1): track 2.49 -> 3.06 mm
- net (no net): vias 2 -> 0
- added copper zone on F.Cu, net /VDD_3V3_SENSORS
- added copper zone on B.Cu, net GND
- added copper zone on F.Cu, net GND
Other:
- board outline added: 19.8 x 16 mm

Commit message: save
Other:
- board text added: "3v3"
- board text added: "BARO_CS"
- board text added: "GND"
- board text added: "ICM_CS"
- board text added: "ICM_DRDY"
- board text added: "Kws 2020-05-29"
- board text added: "MISO"
- board text added: "MOSI"
- board text added: "MPU_CS"
- board text added: "MPU_DRDY"
- board text added: "SCK"
Changed lines of the file:
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@@
   (general
     (thickness 1.6)
-    (drawings 4)
+    (drawings 16)
     (tracks 174)
     (zones 0)
@@
   )
   (setup
-    (last_trace_width 0.2)
+    (last_trace_width 0.25)
     (user_trace_width 0.2)
     (trace_clearance 0.2)
@@
   (module CC0402ZRY5V7BB104:CAPC1005X55N (layer F.Cu)
     (at 141.77 31.29)
-    (fp_text reference C7 (at -1.12 -0.41) (layer F.SilkS)
-      (effects (font (size 0.2 0.2) (thickness 0.05)))
+    (fp_text reference C7 (at -1.15 -0.42) (layer F.SilkS)
+      (effects (font (size 0.4 0.4) (thickness 0.05)))
     )
     (fp_text value 0u1 (at 0.3 0.8) (layer F.Fab)
@@
   (module MPU-9250:QFN40P300X300X105-24N (layer F.Cu)
     (at 138.77 25.41)
-    (fp_text reference U1 (at -1.85 1.9) (layer F.SilkS)
-      (effects (font (size 0.2 0.2) (thickness 0.05)))
+    (fp_text reference U1 (at -1.81 1.92) (layer F.SilkS)
+      (effects (font (size 0.4 0.4) (thickness 0.05)))
     )
     (fp_text value MPU-9250 (at -0.2 2.4) (layer F.Fab)
@@
     (at 141.76 28.73)
     (fp_text reference C6 (at -1.15 -0.44) (layer F.SilkS)
-      (effects (font (size 0.2 0.2) (thickness 0.05)))
+      (effects (font (size 0.4 0.4) (thickness 0.05)))
     )
     (fp_text value 10nF (at 0.3 0.8) (layer F.Fab)
@@
   (module C1608X6S1C225K080AC:CAPC1608X90N (layer F.Cu)
     (at 142.39 30.01)
-    (fp_text reference C8 (at -1.71 -0.59) (layer F.SilkS)
-      (effects (font (size 0.2 0.2) (thickness 0.05)))
+    (fp_text reference C8 (at -1.76 -0.59) (layer F.SilkS)
+      (effects (font (size 0.4 0.4) (thickness 0.05)))
     )
     (fp_text value 2u2 (at -0.3 0.9) (layer F.Fab)
@@
   (module CC0402ZRY5V7BB104:CAPC1005X55N (layer F.Cu)
     (at 143.5 31.31)
-    (fp_text reference C5 (at -0.62 0.69) (layer F.SilkS)
-      (effects (font (size 0.2 0.2) (thickness 0.05)))
+    (fp_text reference C5 (at -0.57 0.75) (layer F.SilkS)
+      (effects (font (size 0.4 0.4) (thickness 0.05)))
     )
     (fp_text value 0u1 (at 0.3 0.8) (layer F.Fab)
@@
   (module SENSOR_CONN:sensorconnect_1x5 (layer F.Cu)
     (at 131.100001 29.2)
-    (fp_text reference J2 (at -1.052001 -6.086) (layer F.SilkS)
-      (effects (font (size 0.2 0.2) (thickness 0.05)))
+    (fp_text reference J2 (at -1.060001 -6.17) (layer F.SilkS)
+      (effects (font (size 0.5 0.5) (thickness 0.05)))
     )
     (fp_text value Conn_01x05 (at -0.1 6.5) (layer F.Fab)
@@
     (at 134.61 25.28 180)
     (fp_text reference C1 (at 1.28 0.73) (layer F.SilkS)
-      (effects (font (size 0.2 0.2) (thickness 0.05)))
+      (effects (font (size 0.4 0.4) (thickness 0.05)))
     )
     (fp_text value 2u2 (at -0.3 0.9) (layer F.Fab)
@@
   (module CC0402ZRY5V7BB104:CAPC1005X55N (layer F.Cu)
     (at 135.23 26.7 180)
-    (fp_text reference C2 (at 0.81 -0.63) (layer F.SilkS)
-      (effects (font (size 0.2 0.2) (thickness 0.05)))
+    (fp_text reference C2 (at 0.86 -0.7) (layer F.SilkS)
+      (effects (font (size 0.4 0.4) (thickness 0.05)))
     )
     (fp_text value 0u1 (at 0.3 0.8) (layer F.Fab)
@@
     (at 138.23 30 180)
     (fp_text reference C3 (at 1.324 0.79) (layer F.SilkS)
-      (effects (font (size 0.2 0.2) (thickness 0.05)))
+      (effects (font (size 0.4 0.4) (thickness 0.05)))
     )
     (fp_text value 2u2 (at -0.3 0.9) (layer F.Fab)
@@
   (module CC0402ZRY5V7BB104:CAPC1005X55N (layer F.Cu)
     (at 135.62 29.78)
-    (fp_text reference C4 (at -0.82 -0.61) (layer F.SilkS)
-      (effects (font (size 0.2 0.2) (thickness 0.05)))
+    (fp_text reference C4 (at -0.92 -0.67) (layer F.SilkS)
+      (effects (font (size 0.4 0.4) (thickness 0.05)))
     )
     (fp_text value 0u1 (at 0.3 0.8) (layer F.Fab)
@@
     (at 145.04 29.24)
     (fp_text reference J1 (at 0.6 -6.38) (layer F.SilkS)
-      (effects (font (size 0.2 0.2) (thickness 0.05)))
+      (effects (font (size 0.4 0.4) (thickness 0.05)))
     )
     (fp_text value Conn_01x06_Male (at 1.6 8.6) (layer F.Fab)
@@
     (tags capacitor)
     (attr smd)
-    (fp_text reference R1 (at 0.764 0.646) (layer F.SilkS)
-      (effects (font (size 0.2 0.2) (thickness 0.05)))
+    (fp_text reference R1 (at 0.77 0.69) (layer F.SilkS)
+      (effects (font (size 0.4 0.4) (thickness 0.05)))
     )
     (fp_text value 220R (at 0 1.17) (layer F.Fab)
@@
   (module MS561101BA03-50:SON125P500X300X100-8N (layer F.Cu)
     (at 137.26 34.08)
-    (fp_text reference U2 (at -1.9 2.58) (layer F.SilkS)
-      (effects (font (size 0.2 0.2) (thickness 0.05)))
+    (fp_text reference U2 (at -1.95 2.59) (layer F.SilkS)
+      (effects (font (size 0.4 0.4) (thickness 0.05)))
     )
     (fp_text value MS561101BA03-50 (at -0.1 3) (layer F.Fab)
@@
     (at 142.6 34.21)
     (fp_text reference U3 (at -2.07 1.62) (layer F.SilkS)
-      (effects (font (size 0.2 0.2) (thickness 0.05)))
+      (effects (font (size 0.4 0.4) (thickness 0.05)))
     )
     (fp_text value ICM-20602 (at 0.3 2.1) (layer F.Fab)
@@
       (rotate (xyz 0 0 0))
     )
+  )
+  (gr_text "Kws\n2020-05-29" (at 131.94 37.14) (layer F.SilkS)
+    (effects (font (size 0.5 0.5) (thickness 0.05)))
+  )
+  (gr_text MPU_CS (at 146.9 25.3) (layer F.SilkS)
+    (effects (font (size 0.4 0.4) (thickness 0.05)))
+  )
+  (gr_text BARO_CS (at 146.9 27.8) (layer F.SilkS)
+    (effects (font (size 0.35 0.35) (thickness 0.05)))
+  )
+  (gr_text ICM_CS (at 146.9 30.3) (layer F.SilkS)
+    (effects (font (size 0.4 0.4) (thickness 0.05)))
+  )
+  (gr_text MPU_DRDY (at 146.9 32.8) (layer F.SilkS)
+    (effects (font (size 0.3 0.3) (thickness 0.05)))
+  )
+  (gr_text ICM_DRDY (at 146.9 35.2) (layer F.SilkS)
+    (effects (font (size 0.3 0.3) (thickness 0.05)))
+  )
+  (gr_text GND (at 146.9 37.7) (layer F.SilkS)
+    (effects (font (size 0.4 0.4) (thickness 0.05)))
+  )
+  (gr_text GND (at 131.2 35.7) (layer F.SilkS)
+    (effects (font (size 0.4 0.4) (thickness 0.05)))
+  )
+  (gr_text MISO (at 131.2 33) (layer F.SilkS)
+    (effects (font (size 0.4 0.4) (thickness 0.05)))
+  )
+  (gr_text MOSI (at 131.2 30.5) (layer F.SilkS)
+    (effects (font (size 0.4 0.4) (thickness 0.05)))
+  )
+  (gr_text SCK (at 131.2 28) (layer F.SilkS)
+    (effects (font (size 0.4 0.4) (thickness 0.05)))
+  )
+  (gr_text "3v3\n" (at 131.2 25.5) (layer F.SilkS)
+    (effects (font (size 0.5 0.5) (thickness 0.05)))
   )
   (gr_line (start 129.25 38) (end 129.25 22) (layer Edge.Cuts) (width 0.05))
@@
   (segment (start 141.3 35.21) (end 141.3 36.33) (width 0.25) (layer F.Cu) (net 5))
   (segment (start 146.87 29.12) (end 144.85 29.12) (width 0.25) (layer F.Cu) (net 5))
+  (segment (start 144.85 29.12) (end 144.84 29.13) (width 0.25) (layer F.Cu) (net 5))
   (via (at 144.84 29.13) (size 0.8) (drill 0.4) (layers F.Cu B.Cu) (net 5))
-  (segment (start 144.85 29.12) (end 144.84 29.13) (width 0.25) (layer F.Cu) (net 5))
-  (segment (start 141.09 32.88) (end 144.84 29.13) (width 0.2) (layer B.Cu) (net 5))
-  (segment (start 141.3 36.33) (end 141.3 32.89) (width 0.2) (layer B.Cu) (net 5))
+  (segment (start 144.84 32.79) (end 141.3 36.33) (width 0.25) (layer B.Cu) (net 5))
+  (segment (start 144.84 29.13) (end 144.84 32.79) (width 0.25) (layer B.Cu) (net 5))
   (segment (start 138.465 34.7) (end 138.46 34.705) (width 0.25) (layer F.Cu) (net 6))
   (via (at 138.122981 28.942888) (size 0.8) (drill 0.4) (layers F.Cu B.Cu) (net 6))
@@
   (segment (start 139.87 34.21) (end 139.605 34.21) (width 0.25) (layer F.Cu) (net 7))
   (segment (start 141.3 34.21) (end 139.87 34.21) (width 0.25) (layer F.Cu) (net 7))
-  (segment (start 139.87 32.984315) (end 139.87 33.55) (width 0.25) (layer B.Cu) (net 7))
-  (segment (start 138.847982 31.962297) (end 139.87 32.984315) (width 0.25) (layer B.Cu) (net 7))
-  (segment (start 137 23.5) (end 138.847982 25.347982) (width 0.25) (layer B.Cu) (net 7))
   (segment (start 131.200001 29.35) (end 133.175 29.35) (width 0.2) (layer F.Cu) (net 7))
   (via (at 133.175 29.35) (size 0.8) (drill 0.4) (layers F.Cu B.Cu) (net 7))
-  (segment (start 137.942867 28.05) (end 138.83 28.05) (width 0.25) (layer B.Cu) (net 7))
-  (segment (start 136.242868 29.749999) (end 137.942867 28.05) (width 0.25) (layer B.Cu) (net 7))
-  (segment (start 133.574999 29.749999) (end 136.242868 29.749999) (width 0.25) (layer B.Cu) (net 7))
-  (segment (start 133.175 29.35) (end 133.574999 29.749999) (width 0.25) (layer B.Cu) (net 7))
-  (segment (start 138.83 28.05) (end 138.847982 31.962297) (width 0.25) (layer B.Cu) (net 7))
-  (segment (start 138.847982 25.347982) (end 138.83 28.05) (width 0.25) (layer B.Cu) (net 7))
+  (segment (start 139.339991 33.019991) (end 139.470001 33.150001) (width 0.25) (layer B.Cu) (net 7))
+  (segment (start 139.470001 33.150001) (end 139.87 33.55) (width 0.25) (layer B.Cu) (net 7))
+  (segment (start 137 23.5) (end 139.339991 25.839991) (width 0.25) (layer B.Cu) (net 7))
+  (segment (start 139.339991 25.839991) (end 139.34 27.74) (width 0.25) (layer B.Cu) (net 7))
+  (segment (start 139.34 27.74) (end 139.339991 33.019991) (width 0.25) (layer B.Cu) (net 7))
+  (segment (start 136.577866 29.415001) (end 138.252867 27.74) (width 0.25) (layer B.Cu) (net 7))
+  (segment (start 138.252867 27.74) (end 139.34 27.74) (width 0.25) (layer B.Cu) (net 7))
+  (segment (start 133.240001 29.415001) (end 136.577866 29.415001) (width 0.25) (layer B.Cu) (net 7))
+  (segment (start 133.175 29.35) (end 133.240001 29.415001) (width 0.25) (layer B.Cu) (net 7))
   (via (at 137.70124 22.787072) (size 0.8) (drill 0.4) (layers F.Cu B.Cu) (net 8))
   (segment (start 138.17 23.865) (end 138.17 23.255832) (width 0.2) (layer F.Cu) (net 8))

Commit message: Sensor board completed
Routing:
- net /BARO_CS: track 19.4 -> 20.1 mm
- net /SPI_INT_MOSI: track 24.8 -> 25.5 mm
Changed lines of the file:
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@@
     (thickness 1.6)
     (drawings 16)
-    (tracks 174)
+    (tracks 177)
     (zones 0)
     (modules 14)
@@
     (45 Margin user hide)
     (46 B.CrtYd user hide)
-    (47 F.CrtYd user)
+    (47 F.CrtYd user hide)
     (48 B.Fab user hide)
     (49 F.Fab user hide)
@@
     (effects (font (size 0.3 0.3) (thickness 0.05)))
   )
-  (gr_text ICM_DRDY (at 146.9 35.2) (layer F.SilkS)
+  (gr_text ICM_DRDY (at 146.88 35.35) (layer F.SilkS)
     (effects (font (size 0.3 0.3) (thickness 0.05)))
   )
@@
   (segment (start 135.66 25.621) (end 135.66 26.7) (width 0.2) (layer F.Cu) (net 1))
   (segment (start 135.319 25.28) (end 135.66 25.621) (width 0.2) (layer F.Cu) (net 1))
-  (segment (start 136.06 32.205) (end 136.06 31.74) (width 0.2) (layer F.Cu) (net 1))
-  (segment (start 136.06 31.74) (end 136.06 31.15) (width 0.2) (layer F.Cu) (net 1))
   (segment (start 141.34 32.5) (end 141.34 31.79) (width 0.2) (layer F.Cu) (net 1))
   (segment (start 141.75 32.91) (end 141.34 32.5) (width 0.2) (layer F.Cu) (net 1))
@@
   (via (at 140.59 30.01) (size 0.8) (drill 0.4) (layers F.Cu B.Cu) (net 1))
   (segment (start 141.681 30.01) (end 140.59 30.01) (width 0.2) (layer F.Cu) (net 1))
-  (segment (start 140.59 26.93518) (end 141.27018 26.255) (width 0.2) (layer B.Cu) (net 1))
-  (segment (start 140.59 30.01) (end 140.59 26.93518) (width 0.2) (layer B.Cu) (net 1))
+  (segment (start 141.670179 28.929821) (end 140.989999 29.610001) (width 0.2) (layer B.Cu) (net 1))
+  (segment (start 140.989999 29.610001) (end 140.59 30.01) (width 0.2) (layer B.Cu) (net 1))
+  (segment (start 141.670179 26.654999) (end 141.670179 28.929821) (width 0.2) (layer B.Cu) (net 1))
+  (segment (start 141.27018 26.255) (end 141.670179 26.654999) (width 0.2) (layer B.Cu) (net 1))
+  (segment (start 136.06 32.205) (end 136.06 31.31) (width 0.25) (layer F.Cu) (net 1))
   (segment (start 142.2 31.024998) (end 143.099 30.125998) (width 0.25) (layer F.Cu) (net 2))
   (segment (start 143.099 30.125998) (end 143.099 30.01) (width 0.25) (layer F.Cu) (net 2))
@@
   (segment (start 146.87 26.62) (end 144.91 26.62) (width 0.25) (layer F.Cu) (net 4))
   (via (at 144.91 26.62) (size 0.8) (drill 0.4) (layers F.Cu B.Cu) (net 4))
-  (segment (start 145.565001 34.524999) (end 142.890001 37.199999) (width 0.25) (layer B.Cu) (net 4))
-  (segment (start 145.565001 27.275001) (end 145.565001 34.524999) (width 0.25) (layer B.Cu) (net 4))
-  (segment (start 138.859999 37.199999) (end 138.46 36.8) (width 0.25) (layer B.Cu) (net 4))
-  (segment (start 142.890001 37.199999) (end 138.859999 37.199999) (width 0.25) (layer B.Cu) (net 4))
-  (segment (start 144.91 26.62) (end 145.565001 27.275001) (width 0.25) (layer B.Cu) (net 4))
+  (segment (start 138.46 36.8) (end 139.08 37.42) (width 0.2) (layer B.Cu) (net 4))
+  (segment (start 139.08 37.42) (end 142.55 37.42) (width 0.2) (layer B.Cu) (net 4))
+  (segment (start 142.55 37.42) (end 146.29 33.68) (width 0.2) (layer B.Cu) (net 4))
+  (segment (start 146.29 28) (end 144.91 26.62) (width 0.2) (layer B.Cu) (net 4))
+  (segment (start 146.29 33.68) (end 146.29 28) (width 0.2) (layer B.Cu) (net 4))
   (via (at 141.3 36.33) (size 0.8) (drill 0.4) (layers F.Cu B.Cu) (net 5))
   (segment (start 141.3 35.21) (end 141.3 36.33) (width 0.25) (layer F.Cu) (net 5))
@@
   (segment (start 131.200001 29.35) (end 133.175 29.35) (width 0.2) (layer F.Cu) (net 7))
   (via (at 133.175 29.35) (size 0.8) (drill 0.4) (layers F.Cu B.Cu) (net 7))
-  (segment (start 139.339991 33.019991) (end 139.470001 33.150001) (width 0.25) (layer B.Cu) (net 7))
-  (segment (start 139.470001 33.150001) (end 139.87 33.55) (width 0.25) (layer B.Cu) (net 7))
-  (segment (start 137 23.5) (end 139.339991 25.839991) (width 0.25) (layer B.Cu) (net 7))
-  (segment (start 139.339991 25.839991) (end 139.34 27.74) (width 0.25) (layer B.Cu) (net 7))
-  (segment (start 139.34 27.74) (end 139.339991 33.019991) (width 0.25) (layer B.Cu) (net 7))
-  (segment (start 136.577866 29.415001) (end 138.252867 27.74) (width 0.25) (layer B.Cu) (net 7))
-  (segment (start 138.252867 27.74) (end 139.34 27.74) (width 0.25) (layer B.Cu) (net 7))
-  (segment (start 133.240001 29.415001) (end 136.577866 29.415001) (width 0.25) (layer B.Cu) (net 7))
+  (segment (start 139.470001 33.150001) (end 139.87 33.55) (width 0.2) (layer B.Cu) (net 7))
+  (segment (start 137 23.5) (end 139.339991 25.839991) (width 0.2) (layer B.Cu) (net 7))
+  (segment (start 139.34 27.74) (end 139.339991 33.019991) (width 0.2) (layer B.Cu) (net 7))
   (segment (start 133.175 29.35) (end 133.240001 29.415001) (width 0.25) (layer B.Cu) (net 7))
+  (segment (start 139.339991 33.019991) (end 139.470001 33.150001) (width 0.2) (layer B.Cu) (net 7))
+  (segment (start 133.574999 29.749999) (end 135.330001 29.749999) (width 0.2) (layer B.Cu) (net 7))
+  (segment (start 133.175 29.35) (end 133.574999 29.749999) (width 0.2) (layer B.Cu) (net 7))
+  (segment (start 138.17 26.91) (end 139.3 26.91) (width 0.2) (layer B.Cu) (net 7))
+  (segment (start 135.330001 29.749999) (end 138.17 26.91) (width 0.2) (layer B.Cu) (net 7))
+  (segment (start 139.339991 25.839991) (end 139.3 26.91) (width 0.2) (layer B.Cu) (net 7))
+  (segment (start 139.3 26.91) (end 139.34 27.74) (width 0.2) (layer B.Cu) (net 7))
   (via (at 137.70124 22.787072) (size 0.8) (drill 0.4) (layers F.Cu B.Cu) (net 8))
   (segment (start 138.17 23.865) (end 138.17 23.255832) (width 0.2) (layer F.Cu) (net 8))
@@
   (via (at 140.19 31.86) (size 0.8) (drill 0.4) (layers F.Cu B.Cu) (net 8))
   (segment (start 140.595001 33.201999) (end 140.186501 32.793499) (width 0.25) (layer F.Cu) (net 8))
-  (segment (start 138.101239 23.187071) (end 137.70124 22.787072) (width 0.25) (layer B.Cu) (net 8))
-  (segment (start 139.790001 31.460001) (end 139.790001 24.875833) (width 0.25) (layer B.Cu) (net 8))
-  (segment (start 139.790001 24.875833) (end 138.101239 23.187071) (width 0.25) (layer B.Cu) (net 8))
-  (segment (start 140.19 31.86) (end 139.790001 31.460001) (width 0.25) (layer B.Cu) (net 8))
+  (segment (start 138.101239 23.187071) (end 137.70124 22.787072) (width 0.2) (layer B.Cu) (net 8))
+  (segment (start 139.790001 31.460001) (end 139.790001 24.875833) (width 0.2) (layer B.Cu) (net 8))
+  (segment (start 139.790001 24.875833) (end 138.101239 23.187071) (width 0.2) (layer B.Cu) (net 8))
+  (segment (start 140.19 31.86) (end 139.790001 31.460001) (width 0.2) (layer B.Cu) (net 8))
   (segment (start 145.42 31.62) (end 146.87 31.62) (width 0.2) (layer F.Cu) (net 15))
   (segment (start 145.350002 31.62) (end 145.42 31.62) (width 0.2) (layer F.Cu) (net 15))
@@
     (polygon
       (pts
-        (xy 149 38) (xy 129.25 38) (xy 129.25 32) (xy 142 32) (xy 142 27.75)
+        (xy 149 38) (xy 129.25 38) (xy 129.236145 32.98) (xy 141.983855 32.98) (xy 142 27.75)
         (xy 139.25 27.75) (xy 139.25 22) (xy 149 22)
       )

Commit message: save sensor
Parts:
- moved U1 0.24 mm to (138.8, 25.7)
Routing:
- net GND: track 24.5 -> 25.6 mm, vias 6 -> 7
- net /SPI_INT_SCK: track 25.4 -> 26.3 mm
- net /VDD_3V3_SENSORS: track 21.4 -> 21.9 mm
